Commit message: feat: add the 3D playback of the trajectory solve in the browser
meshcat shows the robot following q_cmd with the target and solved TCP paths after a
solve. The Marvin meshes move into robots/marvin/meshes (LFS) with relative paths in
the URDF, and the image gains meshcat.

File: robots/marvin/urdf/serial_marvin_with_gripper.urdf (robot description, URDF)
Before this commit: robot serial_marvin_with_gripper, 40 links, 39 joints
Links:
- link Base_L: geometry collision mesh filename=../meshes/marvin/Base_L.STL; visual mesh filename=../meshes/marvin/Base_L.STL
- link Base_R: geometry collision mesh filename=../meshes/marvin/Base_R.STL; visual mesh filename=../meshes/marvin/Base_R.STL
- link Link1_L: geometry collision mesh filename=../meshes/marvin/Link1_L.STL; visual mesh filename=../meshes/marvin/Link1_L.STL
- link Link1_R: geometry collision mesh filename=../meshes/marvin/Link1_R.STL; visual mesh filename=../meshes/marvin/Link1_R.STL
- link Link2_L: geometry collision mesh filename=../meshes/marvin/Link2_L.STL; visual mesh filename=../meshes/marvin/Link2_L.STL
- link Link2_R: geometry collision mesh filename=../meshes/marvin/Link2_R.STL; visual mesh filename=../meshes/marvin/Link2_R.STL
- link Link3_L: geometry collision mesh filename=../meshes/marvin/Link3_L.STL; visual mesh filename=../meshes/marvin/Link3_L.STL
- link Link3_R: geometry collision mesh filename=../meshes/marvin/Link3_R.STL; visual mesh filename=../meshes/marvin/Link3_R.STL
- link Link4_L: geometry collision mesh filename=../meshes/marvin/Link4_L.STL; visual mesh filename=../meshes/marvin/Link4_L.STL
- link Link4_R: geometry collision mesh filename=../meshes/marvin/Link4_R.STL; visual mesh filename=../meshes/marvin/Link4_R.STL
- link Link5_L: geometry collision mesh filename=../meshes/marvin/Link5_L.STL; visual mesh filename=../meshes/marvin/Link5_L.STL
- link Link5_R: geometry collision mesh filename=../meshes/marvin/Link5_R.STL; visual mesh filename=../meshes/marvin/Link5_R.STL
- link Link6_L: geometry collision mesh filename=../meshes/marvin/Link6_L.STL; visual mesh filename=../meshes/marvin/Link6_L.STL
- link Link6_R: geometry collision mesh filename=../meshes/marvin/Link6_R.STL; visual mesh filename=../meshes/marvin/Link6_R.STL
- link Link7_L: geometry collision mesh filename=../meshes/marvin/Link7_L.STL; visual mesh filename=../meshes/marvin/Link7_L.STL
- link Link7_R: geometry collision mesh filename=../meshes/marvin/Link7_R.STL; visual mesh filename=../meshes/marvin/Link7_R.STL
- link Link_Base: geometry collision mesh filename=../meshes/marvin/Link_Base.STL; visual mesh filename=../meshes/marvin/Link_Base.STL
- link Link_Stand: geometry collision mesh filename=../meshes/marvin/Link_Stand.STL; visual mesh filename=../meshes/marvin/Link_Stand.STL
- link left_flange: geometry collision mesh filename=../meshes/marvin/flange.STL; visual mesh filename=../meshes/marvin/flange.STL
- link left_gripper_f90c_base_link: geometry collision mesh filename=../meshes/gripper_f90c/gripper_f90c_base_link.STL; visual mesh filename=../meshes/gripper_f90c/gripper_f90c_base_link.STL
- link left_gripper_f90c_left_1_link: geometry collision mesh filename=../meshes/gripper_f90c/gripper_f90c_left_1_link.STL; visual mesh filename=../meshes/gripper_f90c/gripper_f90c_left_1_link.STL
- link left_gripper_f90c_left_2_link: geometry collision mesh filename=../meshes/gripper_f90c/gripper_f90c_left_2_link.STL; visual mesh filename=../meshes/gripper_f90c/gripper_f90c_left_2_link.STL
- link left_gripper_f90c_left_pad_link: geometry collision mesh filename=../meshes/gripper_f90c/gripper_f90c_left_pad_link.STL; visual mesh filename=../meshes/gripper_f90c/gripper_f90c_left_pad_link.STL
- link left_gripper_f90c_left_support_link: geometry collision mesh filename=../meshes/gripper_f90c/gripper_f90c_left_support_link.STL; visual mesh filename=../meshes/gripper_f90c/gripper_f90c_left_support_link.STL
- link left_gripper_f90c_right_1_link: geometry collision mesh filename=../meshes/gripper_f90c/gripper_f90c_right_1_link.STL; visual mesh filename=../meshes/gripper_f90c/gripper_f90c_right_1_link.STL
- link left_gripper_f90c_right_2_link: geometry collision mesh filename=../meshes/gripper_f90c/gripper_f90c_right_2_link.STL; visual mesh filename=../meshes/gripper_f90c/gripper_f90c_right_2_link.STL
- link left_gripper_f90c_right_pad_link: geometry collision mesh filename=../meshes/gripper_f90c/gripper_f90c_right_pad_link.STL; visual mesh filename=../meshes/gripper_f90c/gripper_f90c_right_pad_link.STL
- link left_gripper_f90c_right_support_link: geometry collision mesh filename=../meshes/gripper_f90c/gripper_f90c_right_support_link.STL; visual mesh filename=../meshes/gripper_f90c/gripper_f90c_right_support_link.STL
- link right_flange: geometry collision mesh filename=../meshes/marvin/flange.STL; visual mesh filename=../meshes/marvin/flange.STL
- link right_gripper_f90c_base_link: geometry collision mesh filename=../meshes/gripper_f90c/gripper_f90c_base_link.STL; visual mesh filename=../meshes/gripper_f90c/gripper_f90c_base_link.STL
- link right_gripper_f90c_left_1_link: geometry collision mesh filename=../meshes/gripper_f90c/gripper_f90c_left_1_link.STL; visual mesh filename=../meshes/gripper_f90c/gripper_f90c_left_1_link.STL
- link right_gripper_f90c_left_2_link: geometry collision mesh filename=../meshes/gripper_f90c/gripper_f90c_left_2_link.STL; visual mesh filename=../meshes/gripper_f90c/gripper_f90c_left_2_link.STL
- link right_gripper_f90c_left_pad_link: geometry collision mesh filename=../meshes/gripper_f90c/gripper_f90c_left_pad_link.STL; visual mesh filename=../meshes/gripper_f90c/gripper_f90c_left_pad_link.STL
- link right_gripper_f90c_left_support_link: geometry collision mesh filename=../meshes/gripper_f90c/gripper_f90c_left_support_link.STL; visual mesh filename=../meshes/gripper_f90c/gripper_f90c_left_support_link.STL
- link right_gripper_f90c_right_1_link: geometry collision mesh filename=../meshes/gripper_f90c/gripper_f90c_right_1_link.STL; visual mesh filename=../meshes/gripper_f90c/gripper_f90c_right_1_link.STL
- link right_gripper_f90c_right_2_link: geometry collision mesh filename=../meshes/gripper_f90c/gripper_f90c_right_2_link.STL; visual mesh filename=../meshes/gripper_f90c/gripper_f90c_right_2_link.STL
- link right_gripper_f90c_right_pad_link: geometry collision mesh filename=../meshes/gripper_f90c/gripper_f90c_right_pad_link.STL; visual mesh filename=../meshes/gripper_f90c/gripper_f90c_right_pad_link.STL
- link right_gripper_f90c_right_support_link: geometry collision mesh filename=../meshes/gripper_f90c/gripper_f90c_right_support_link.STL; visual mesh filename=../meshes/gripper_f90c/gripper_f90c_right_support_link.STL
